Commit message: Atualizando e recuperando dados antes do bug

File: bicopter_description/urdf/bicopter_ass.xacro (robot description, xacro)
@@ -46,5 +46,5 @@
    <xacro:tilt prefix="right" reflect="-1" />
    <xacro:tilt prefix="left" reflect="1" />
-   <!-- CRIACAO DOS STATOR E SUAS JUNTAS (JOINTS) -->
+   <!-- CRIACAO DOS STATOR E SUAS JUNTAS (JOINTS)  -->
    <xacro:stator prefix="right" reflect="-1" parent="right_tilt"/>
    <xacro:stator prefix="left"  reflect="1" parent="left_tilt" />

File: bicopter_description/urdf/bicopter_base.xacro (robot description, xacro)
@@ -14,6 +14,11 @@
   <!-- MACRO PARA CRIACAO DA BASE DO BICOPTER -->
   <xacro:macro name="bicopter_base">
+  <!---->
   <link name="base_link">
   </link>
+  <joint name="base_joint" type="fixed">
+    <parent link="base_link"/>
+    <child link="base_link_inertial"/>
+  </joint>
   <link name="base_link_inertial">
     <visual>
@@ -31,8 +36,4 @@
     <xacro:default_inertial mass="0.1419" ixx="0.1942e-6" ixy="0" ixz="0" iyy="0.3362e-6" iyz="-0.0021e-6" izz="0.5259e-6"/>
   </link>
-  <joint name="base_joint" type="fixed">
-    <parent link="base_link"/>
-    <child link="base_link_inertial"/>
-  </joint>
   <!-- attach multirotor_base_plugin to the base_link -->
   <gazebo>
@@ -254,48 +255,4 @@
     </gazebo>
   </xacro:macro>
-  <!--XACRO DO IMU : joint , link , sensor
-  <xacro:macro name="imu_sensor" params="xyz rpy parent">
-    <link name="imu_sensor_link">
-        <collision>
-            <origin xyz="0 0 0" rpy="0 0 0"/>
-            <geometry>
-                <box size="0.02 0.02 0.01"/>
-            </geometry>
-        </collision>
-        <visual>
-            <geometry>
-                <box size="0.02 0.02 0.01"/>
-            </geometry>
-            <origin xyz="0 0 0" rpy="0 0 0"/>
-             <material name="blue"/>
-        </visual>
-        <inertial>
-            <mass value="0.001" />
-            <origin xyz="0 0 0" rpy="0 0 0"/>
-            <inertia ixx="0.00000015" ixy="0" ixz="0" iyy="0.00000015" iyz="0" izz="0.00000015" />
-        </inertial>
-    </link>
-    <joint name="imu_sensor_joint" type="fixed">
-        <axis xyz="0 0 1" />
-        <origin xyz="${xyz}" rpy="${rpy}"/>
-        <parent link="${parent}"/>
-        <child link="imu_sensor_link"/>
-    </joint>
-    <gazebo>
-        <plugin name='imu_plugin' filename='libgazebo_ros_imu.so'>
-              <always_on>1</always_on>
-              <topicName>imu_data</topicName>
-              <bodyName>imu_sensor_link</bodyName>
-              <updateRateHZ>10.0</updateRateHZ>
-              <gaussianNoise>0.0</gaussianNoise>
-              <xyzOffset>0 0 0</xyzOffset>
-              <rpyOffset>0 0 0</rpyOffset>
-        </plugin>
-    </gazebo>
-  </xacro:macro>
-   -->
-     <!-- CRIACAO DOS IMU
-   <xacro:imu_sensor xyz="0 0.05 0" rpy="0 0 0" parent="base_link" />
-   -->
   <!--MACRO PARA CRIACAO DO ROTOR -->
   <xacro:macro name="vertical_rotor" params="prefix direction motor_constant moment_constant parent mass_rotor radius_rotor time_constant_up time_constant_down max_rot_velocity motor_number rotor_drag_coefficient rolling_moment_coefficient color mesh mesh_scale *origin *inertia">
@@ -307,7 +264,4 @@
     </joint>
     -->
-    <!-- TODO(ff): not currently set because it's not yet supported -->
-    <!-- <gazebo reference="rotor_${motor_number}_joint"> <axis> <xyz>0 0 1</xyz>
-      <limit> <velocity> ${max_rot_velocity} </velocity> </limit> </axis> </gazebo> -->
     <link name="${prefix}_rotor">
       <inertial>
@@ -361,4 +315,5 @@
       </plugin>
     </gazebo>
+    <!-- -->
     <gazebo reference="${prefix}_rotor">
       <material>Gazebo/${color}</material>
@@ -366,2 +321,46 @@
     </xacro:macro>
  </robot>
+ <!--XACRO DO IMU : joint , link , sensor
+  <xacro:macro name="imu_sensor" params="xyz rpy parent">
+    <link name="imu_sensor_link">
+        <collision>
+            <origin xyz="0 0 0" rpy="0 0 0"/>
+            <geometry>
+                <box size="0.02 0.02 0.01"/>
+            </geometry>
+        </collision>
+        <visual>
+            <geometry>
+                <box size="0.02 0.02 0.01"/>
+            </geometry>
+            <origin xyz="0 0 0" rpy="0 0 0"/>
+             <material name="blue"/>
+        </visual>
+        <inertial>
+            <mass value="0.001" />
+            <origin xyz="0 0 0" rpy="0 0 0"/>
+            <inertia ixx="0.00000015" ixy="0" ixz="0" iyy="0.00000015" iyz="0" izz="0.00000015" />
+        </inertial>
+    </link>
+    <joint name="imu_sensor_joint" type="fixed">
+        <axis xyz="0 0 1" />
+        <origin xyz="${xyz}" rpy="${rpy}"/>
+        <parent link="${parent}"/>
+        <child link="imu_sensor_link"/>
+    </joint>
+    <gazebo>
+        <plugin name='imu_plugin' filename='libgazebo_ros_imu.so'>
+              <always_on>1</always_on>
+              <topicName>imu_data</topicName>
+              <bodyName>imu_sensor_link</bodyName>
+              <updateRateHZ>10.0</updateRateHZ>
+              <gaussianNoise>0.0</gaussianNoise>
+              <xyzOffset>0 0 0</xyzOffset>
+              <rpyOffset>0 0 0</rpyOffset>
+        </plugin>
+    </gazebo>
+  </xacro:macro>
+   -->
+     <!-- CRIACAO DOS IMU
+   <xacro:imu_sensor xyz="0 0.05 0" rpy="0 0 0" parent="base_link" />
+   -->

Commit message: Parando a simulaçao e encontrando o estranho defeito

File: bicopter_description/urdf/bicopter_ass.xacro (robot description, xacro)
@@ -70,4 +70,5 @@
     <xacro:insert_block name="rotor_inertia" />
   </xacro:vertical_rotor>
+   <!-- -->
    <xacro:vertical_rotor
     prefix="right"

File: bicopter_description/urdf/bicopter_assembly.xacro (robot description, xacro)
@@ -19,5 +19,5 @@
   <!-- Included URDF Files -->
   <xacro:include filename="$(find bicopter_sim)/bicopter_description/urdf/bicopter_base.xacro" />
-   <!-- inertia of a single rotor, assuming it is a cuboid. Height=3mm, width=15mm -->
+   <!-- inertia of a single rotor, assuming it is a cuboid. Height=3mm, width=15mm
   <xacro:property name="rotor_inertia">
     <inertia
@@ -25,6 +25,15 @@
     iyy="${1/12 * mass_rotor * (4 * radius_rotor * radius_rotor + 0.003 * 0.003) * rotor_velocity_slowdown_sim}"
     izz="${1/12 * mass_rotor * (4 * radius_rotor * radius_rotor + 0.015 * 0.015) * rotor_velocity_slowdown_sim}"
-    ixy="0.0" ixz="0.0"  iyz="0.0" /> <!-- [kg.m^2] [kg.m^2] [kg.m^2] [kg.m^2] [kg.m^2] [kg.m^2] -->
+    ixy="0.0" ixz="0.0"  iyz="0.0" />
+  </xacro:property> -->
+  <!-- -->
+  <xacro:property name="rotor_inertia">
+    <inertia
+    ixx="${1/12 * mass_rotor * (0.015 * 0.015 + 0.003 * 0.003)}"
+    iyy="${1/12 * mass_rotor * (4 * radius_rotor * radius_rotor + 0.003 * 0.003)}"
+    izz="${1/12 * mass_rotor * (4 * radius_rotor * radius_rotor + 0.015 * 0.015)}"
+    ixy="0.0" ixz="0.0"  iyz="0.0" />
   </xacro:property>
+  <!-- [kg.m^2] [kg.m^2] [kg.m^2] [kg.m^2] [kg.m^2] [kg.m^2] -->
   <xacro:bicopter_base/>
    <!-- CRIACAO DOS MANCAIS E SUAS JUNTAS (JOINTS) -->

File: bicopter_description/urdf/bicopter_base.xacro (robot description, xacro)
@@ -297,4 +297,5 @@
       </joint>
     </transmission>
+    <!--
     <gazebo>
       <plugin name="${prefix}_motor_model" filename="librotors_gazebo_motor_model.so">
@@ -315,5 +316,5 @@
       </plugin>
     </gazebo>
-    <!-- -->
+     -->
     <gazebo reference="${prefix}_rotor">
       <material>Gazebo/${color}</material>
