Commit message: Tornando a rotor joint fixa e limitando o angulo de tilt para evitar colisao com o solo

File: bicopter_description/urdf/bicopter_base.xacro (robot description, xacro)
@@ -257,11 +257,10 @@
   <!--MACRO PARA CRIACAO DO ROTOR -->
   <xacro:macro name="vertical_rotor" params="prefix direction motor_constant moment_constant parent mass_rotor radius_rotor time_constant_up time_constant_down max_rot_velocity motor_number rotor_drag_coefficient rolling_moment_coefficient color mesh mesh_scale *origin *inertia">
-    <!--
-    <joint name="rotor_${motor_number}_joint" type="fixed">
+    <!-- -->
+    <joint name="${prefix}_rotor_joint" type="fixed">
       <xacro:insert_block name="origin" />
       <parent link="${parent}" />
-      <child link="rotor_${motor_number}" />
-    </joint>
-    -->
+      <child link="${prefix}_rotor" />
+    </joint>
     <link name="${prefix}_rotor">
       <inertial>
@@ -280,5 +279,5 @@
       </collision>
     </link>
-     <!-- Rotor joint and link  -->
+     <!-- Rotor joint and link
     <joint name="${prefix}_rotor_joint" type="continuous">
       <xacro:insert_block name="origin" />
@@ -297,4 +296,5 @@
       </joint>
     </transmission>
+    -->
     <!--
     <gazebo>
