Commit message: Realizando a implementacao como o tutorial de Wil Selby

File: bicopter_description/urdf/structure_base.xacro (robot description, xacro)
@@ -13,5 +13,5 @@
   </xacro:macro>
   <!-- MACRO PARA CRIACAO DA BASE DO BICOPTER -->
-  <xacro:macro name="bicopter_base">
+  <xacro:macro name="bicopter_base" params="robot_namespace">
   <!---->
   <link name="base_link">
@@ -39,6 +39,7 @@
   <gazebo>
     <plugin filename="librotors_gazebo_multirotor_base_plugin.so" name="rosbag">
-      <linkName>base_link</linkName>
-      <rotorVelocitySlowdownSim>${rotor_velocity_slowdown_sim}</rotorVelocitySlowdownSim>
+      <robotNamespace>${robot_namespace}</robotNamespace>
+        <linkName>base_link</linkName>
+        <rotorVelocitySlowdownSim>${rotor_velocity_slowdown_sim}</rotorVelocitySlowdownSim>
     </plugin>
   </gazebo>
@@ -256,12 +257,19 @@
   </xacro:macro>
   <!--MACRO PARA CRIACAO DO ROTOR -->
-  <xacro:macro name="vertical_rotor" params="prefix direction motor_constant moment_constant parent mass_rotor radius_rotor time_constant_up time_constant_down max_rot_velocity motor_number rotor_drag_coefficient rolling_moment_coefficient color mesh mesh_scale *origin *inertia">
-    <!-- -->
-    <joint name="${prefix}_rotor_joint" type="fixed">
+  <!-- Rotor joint and link -->
+  <xacro:macro name="vertical_rotor"
+    params="robot_namespace suffix direction motor_constant moment_constant parent mass_rotor radius_rotor time_constant_up time_constant_down max_rot_velocity motor_number rotor_drag_coefficient rolling_moment_coefficient color mesh mesh_scale *origin *inertia">
+    <joint name="rotor_${motor_number}_joint" type="continuous">
       <xacro:insert_block name="origin" />
+      <axis xyz="0 0 1" />
+      <!-- TODO(ff): not currently set because it's not yet supported -->
+      <!-- <limit effort="2000" velocity="${max_rot_velocity}" /> -->
       <parent link="${parent}" />
-      <child link="${prefix}_rotor" />
-    </joint>
-    <link name="${prefix}_rotor">
+      <child link="rotor_${motor_number}" />
+    </joint>
+    <!-- TODO(ff): not currently set because it's not yet supported -->
+    <!-- <gazebo reference="rotor_${motor_number}_joint"> <axis> <xyz>0 0 1</xyz>
+      <limit> <velocity> ${max_rot_velocity} </velocity> </limit> </axis> </gazebo> -->
+    <link name="rotor_${motor_number}">
       <inertial>
         <mass value="${mass_rotor}" /> <!-- [kg] -->
@@ -270,5 +278,9 @@
       <visual>
         <geometry>
-          <mesh filename="package://bicopter_sim/bicopter_description/meshes/${mesh}_${direction}.dae" scale="${mesh_scale}" />
+          <!-- <cylinder length="0.005" radius="${radius_rotor}"/> --> <!-- [m] -->
+          <!-- <mesh filename="package://rotors_description/meshes/propeller_${direction}.dae" -->
+          <mesh filename="package://bicopter_sim/bicopter_description/meshes/${mesh}_${direction}.dae"
+            scale="${mesh_scale}" />
+          <!-- <box size="${2*radius_rotor} 0.01 0.005"/> -->
         </geometry>
       </visual>
@@ -279,27 +291,9 @@
       </collision>
     </link>
-     <!-- Rotor joint and link
-    <joint name="${prefix}_rotor_joint" type="continuous">
-      <xacro:insert_block name="origin" />
-      <axis xyz="0 0 1" />
-      <limit effort="1000" velocity="1.0"/>
-      <parent link="${parent}" />
-      <child link="${prefix}_rotor" />
-    </joint>
-    <transmission name="${prefix}_motor_trans" type="SimpleTransmission">
-      <type>transmission_interface/SimpleTransmission</type>
-      <actuator name="${prefix}_motor">
-        <mechanicalReduction>1</mechanicalReduction>
-      </actuator>
-      <joint name="${prefix}_rotor_joint">
-        <hardwareInterface>hardware_interface/PositionJointInterface</hardwareInterface>
-      </joint>
-    </transmission>
-    -->
-    <!--
     <gazebo>
-      <plugin name="${prefix}_motor_model" filename="librotors_gazebo_motor_model.so">
-        <jointName>${prefix}_rotor_joint</jointName>
-        <linkName>${prefix}_rotor</linkName>
+      <plugin name="${suffix}_motor_model" filename="librotors_gazebo_motor_model.so">
+        <robotNamespace>${robot_namespace}</robotNamespace>
+        <jointName>rotor_${motor_number}_joint</jointName>
+        <linkName>rotor_${motor_number}</linkName>
         <turningDirection>${direction}</turningDirection>
         <timeConstantUp>${time_constant_up}</timeConstantUp>
@@ -312,13 +306,12 @@
         <rotorDragCoefficient>${rotor_drag_coefficient}</rotorDragCoefficient>
         <rollingMomentCoefficient>${rolling_moment_coefficient}</rollingMomentCoefficient>
-        <motorSpeedPubTopic>motor_speed/${prefix}</motorSpeedPubTopic>
+        <motorSpeedPubTopic>motor_speed/${motor_number}</motorSpeedPubTopic>
         <rotorVelocitySlowdownSim>${rotor_velocity_slowdown_sim}</rotorVelocitySlowdownSim>
       </plugin>
     </gazebo>
-     -->
-    <gazebo reference="${prefix}_rotor">
+    <gazebo reference="rotor_${motor_number}">
       <material>Gazebo/${color}</material>
     </gazebo>
-    </xacro:macro>
+  </xacro:macro>
  </robot>
  <!--XACRO DO IMU : joint , link , sensor

File: tutorial/urdf/bicopter_base.xacro (robot description, xacro)
@@ -13,8 +13,13 @@
   </xacro:macro>
   <!-- MACRO PARA CRIACAO DA BASE DO BICOPTER -->
-  <xacro:macro name="bicopter_base" params="robot_namespace">
-  <link name="${robot_namespace}/base_link">
+  <xacro:macro name="bicopter_base">
+  <!---->
+  <link name="base_link">
   </link>
-  <link name="${robot_namespace}/base_link_inertial">
+  <joint name="base_joint" type="fixed">
+    <parent link="base_link"/>
+    <child link="base_link_inertial"/>
+  </joint>
+  <link name="base_link_inertial">
     <visual>
       <origin rpy="0 0 0" xyz="0 0 0"/>
@@ -31,13 +36,8 @@
     <xacro:default_inertial mass="0.1419" ixx="0.1942e-6" ixy="0" ixz="0" iyy="0.3362e-6" iyz="-0.0021e-6" izz="0.5259e-6"/>
   </link>
-  <joint name="${robot_namespace}/base_joint" type="fixed">
-    <parent link="${robot_namespace}/base_link"/>
-    <child link="${robot_namespace}/base_link_inertial"/>
-  </joint>
   <!-- attach multirotor_base_plugin to the base_link -->
   <gazebo>
     <plugin filename="librotors_gazebo_multirotor_base_plugin.so" name="rosbag">
-      <robotNamespace>${robot_namespace}</robotNamespace>
-      <linkName>${robot_namespace}/base_link</linkName>
+      <linkName>base_link</linkName>
       <rotorVelocitySlowdownSim>${rotor_velocity_slowdown_sim}</rotorVelocitySlowdownSim>
     </plugin>
@@ -45,6 +45,6 @@
   </xacro:macro>
   <!-- MACRO PARA CRIACAO DO MANCAL -->
-  <xacro:macro name="mancal" params="robot_namespace prefix reflect">
-    <link name="${robot_namespace}/${prefix}_mancal">
+  <xacro:macro name="mancal" params="prefix reflect">
+    <link name="${prefix}_mancal">
       <visual>
         <geometry>
@@ -61,13 +61,13 @@
       <xacro:default_inertial mass="0.01971" ixx="3.0541067e-09" ixy="-1.22135e-11" ixz="2.8446e-12" iyy="3.361632324e-07" iyz="-2.06933e-09" izz="5.258915527e-07"/>
     </link>
-    <joint name="${robot_namespace}/base_to_${prefix}_mancal" type="fixed">
-      <parent link="${robot_namespace}/base_link"/>
-      <child link="${robot_namespace}/${prefix}_mancal"/>
+    <joint name="base_to_${prefix}_mancal" type="fixed">
+      <parent link="base_link"/>
+      <child link="${prefix}_mancal"/>
       <origin xyz="${reflect*0.07} 0 0.0142" />
     </joint>
   </xacro:macro>
   <!-- MACRO PARA CRIACAO DO TUBE ARM -->
-  <xacro:macro name="tube_arm" params="robot_namespace prefix reflect">
-    <link name="${robot_namespace}/${prefix}_tube_arm">
+  <xacro:macro name="tube_arm" params="prefix reflect">
+    <link name="${prefix}_tube_arm">
       <visual>
         <geometry>
@@ -84,13 +84,13 @@
       <xacro:default_inertial mass="0.03022" ixx="1.7960983e-09" ixy="-2.3981262e-09" ixz="-2.08e-14" iyy="2.15995621e-08" iyz="-7.0e-16" izz="2.17520676e-08"/>
     </link>
-    <joint name="${robot_namespace}/base_to_${prefix}_tube_arm" type="fixed">
-      <parent link="${robot_namespace}/base_link"/>
-      <child link="${robot_namespace}/${prefix}_tube_arm"/>
+    <joint name="base_to_${prefix}_tube_arm" type="fixed">
+      <parent link="base_link"/>
+      <child link="${prefix}_tube_arm"/>
       <origin xyz="${reflect*0.115} 0 0.0142" />
     </joint>
   </xacro:macro>
   <!-- MACRO PARA CRIACAO DO ARM -->
-   <xacro:macro name="arm" params="robot_namespace prefix releve reflect">
-    <link name="${robot_namespace}/${prefix}_arm">
+   <xacro:macro name="arm" params="prefix releve reflect">
+    <link name="${prefix}_arm">
       <visual>
         <geometry>
@@ -107,13 +107,13 @@
       <xacro:default_inertial mass="0.03133" ixx="4.021067e-09" ixy="2.7460985e-09" ixz="-1.840184e-10" iyy="3.54965027e-08" iyz="-7.66613e-11" izz="3.39598694e-08"/>
     </link>
-    <joint name="${robot_namespace}/base_to_${prefix}_arm" type="fixed">
-      <parent link="${robot_namespace}/${prefix}_tube_arm"/>
-      <child link="${robot_namespace}/${prefix}_arm"/>
+    <joint name="base_to_${prefix}_arm" type="fixed">
+      <parent link="${prefix}_tube_arm"/>
+      <child link="${prefix}_arm"/>
       <origin xyz="${reflect*0.1} ${reflect*-0.022} 0"/>
     </joint>
   </xacro:macro>
   <!-- MACRO PARA CRIACAO DO ARM2 -->
-   <xacro:macro name="arm2" params="robot_namespace prefix releve reflect">
-    <link name="${robot_namespace}/${prefix}_arm2">
+   <xacro:macro name="arm2" params="prefix releve reflect">
+    <link name="${prefix}_arm2">
       <visual>
         <geometry>
@@ -130,13 +130,13 @@
       <xacro:default_inertial mass="0.01847" ixx="3.201813e-10" ixy="0.00" ixz="0.00" iyy="5.4531342e-09" iyz="0.00" izz="5.4531342e-09"/>
     </link>
-    <joint name="${robot_namespace}/base_to_${prefix}_arm2" type="fixed">
-      <parent link="${robot_namespace}/${prefix}_tube_arm"/>
-      <child link="${robot_namespace}/${prefix}_arm2"/>
+    <joint name="base_to_${prefix}_arm2" type="fixed">
+      <parent link="${prefix}_tube_arm"/>
+      <child link="${prefix}_arm2"/>
       <origin xyz="${reflect*0.1} ${reflect*0.03} 0"/>
     </joint>
   </xacro:macro>
    <!-- MACRO PARA CRIACAO DO LEG -->
-   <xacro:macro name="leg" params="robot_namespace prefix reflect">
-    <link name="${robot_namespace}/${prefix}_leg">
+   <xacro:macro name="leg" params="prefix reflect">
+    <link name="${prefix}_leg">
       <visual>
         <geometry>
@@ -153,10 +153,10 @@
       <xacro:default_inertial mass="0.00823" ixx="1.91376434e-08" ixy="7.0e-16" ixz="-2.0e-16" iyy="4.2566975e-09" iyz="-1.0e-15" izz="1.49469467e-08"/>
     </link>
-    <joint name="${robot_namespace}/base_to_${prefix}_leg" type="fixed">
-      <parent link="${robot_namespace}/base_link"/>
-      <child link="${robot_namespace}/${prefix}_leg"/>
+    <joint name="base_to_${prefix}_leg" type="fixed">
+      <parent link="base_link"/>
+      <child link="${prefix}_leg"/>
       <origin xyz="${reflect*0.035} 0.0075 -0.0025"/>
     </joint>
-    <gazebo reference="${robot_namespace}/${prefix}_leg">
+    <gazebo reference="${prefix}_leg">
       <mu1 value="200.0"/>
       <mu2 value="100.0"/>
@@ -166,6 +166,6 @@
   </xacro:macro>
    <!-- MACRO PARA CRIACAO DO TILT E SUAS TRANSMISSOES-->
-   <xacro:macro name="tilt" params="robot_namespace prefix reflect">
-    <link name="${robot_namespace}/${prefix}_tilt">
+   <xacro:macro name="tilt" params="prefix reflect">
+    <link name="${prefix}_tilt">
       <visual>
         <geometry>
@@ -176,26 +176,34 @@
       <collision>
         <geometry>
-          <cylinder length="0.02" radius="0.02"/>
-        </geometry>
-      <origin rpy="0 0 0" xyz="0 0 0"/>
+          <cylinder length="0.005" radius="0.02"/>
+        </geometry>
+      <origin rpy="0 0 0" xyz="0 0 -0.01"/>
       </collision>
       <xacro:default_inertial mass="0.00526" ixx="1.8322357e-09" ixy="2.628e-13" ixz="4.879e-13" iyy="3.454043e-10" iyz="-2.906790e-11" izz="1.9750971e-09"/>
     </link>
-    <joint name="${robot_namespace}/arm_to_${prefix}_tilt" type="revolute">
+    <joint name="arm_to_${prefix}_tilt" type="revolute">
       <axis xyz="0 ${reflect*1} 0"/>
       <limit effort="1000.0" lower="0.0" upper="${pi/2}" velocity="0.5"/>
       <origin rpy="0 0 0" xyz="0 ${reflect*0.02} 0"/>
-      <parent link="${robot_namespace}/${prefix}_arm"/>
-      <child link="${robot_namespace}/${prefix}_tilt"/>
+      <parent link="${prefix}_arm"/>
+      <child link="${prefix}_tilt"/>
       <origin xyz="${reflect*0.035} ${reflect*0.0075} -0.0025"/>
     </joint>
+    <!--
+    <joint name="arm_to_${prefix}_tilt" type="fixed">
+      <origin rpy="0 0 0" xyz="0 ${reflect*0.02} 0"/>
+      <parent link="${prefix}_arm"/>
+      <child link="${prefix}_tilt"/>
+      <origin xyz="${reflect*0.035} ${reflect*0.0075} -0.0025"/>
+    </joint>
+    -->
      <!-- This block connects the tilt_rotor joint to an actuator (motor), which informs both
   simulation and visualization of the robot -->
-    <transmission name="${robot_namespace}/${prefix}_tilt_trans" type="SimpleTransmission">
+    <transmission name="${prefix}_tilt_trans" type="SimpleTransmission">
       <type>transmission_interface/SimpleTransmission</type>
-      <actuator name="${robot_namespace}/${prefix}_tilt_motor">
+      <actuator name="${prefix}_tilt_motor">
         <mechanicalReduction>1</mechanicalReduction>
       </actuator>
-      <joint name="${robot_namespace}/arm_to_${prefix}_tilt">
+      <joint name="arm_to_${prefix}_tilt">
         <hardwareInterface>hardware_interface/PositionJointInterface</hardwareInterface>
       </joint>
@@ -203,6 +211,6 @@
   </xacro:macro>
   <!-- MACRO PARA CRIACAO DO ESTATOR -->
-   <xacro:macro name="stator" params="robot_namespace prefix">
-    <link name="${robot_namespace}/${prefix}_stator">
+   <xacro:macro name="stator" params="prefix reflect parent">
+    <link name="${prefix}_stator">
       <visual>
         <geometry>
@@ -215,18 +223,104 @@
          <cylinder length="0.035" radius="0.014"/>
         </geometry>
-        <origin rpy="0 0 0" xyz="0 0 0.009"/>
+        <origin rpy="0 0 0" xyz="0 0 0.011"/>
       </collision>
       <xacro:default_inertial mass="0.053" ixx="${(1/12)*0.053*(3*0.014*0.014+0.035*0.035)}" ixy="0.00" ixz="0.00" iyy="${(1/12)*0.053*(3*0.014*0.014+0.035*0.035)}" iyz="0.00" izz="${(1/2)*0.053*(0.014*0.014)}"/>
     </link>
-    <joint name="${robot_namespace}/tilt_to_${prefix}_stator" type="fixed">
-      <parent link="${robot_namespace}/${prefix}_tilt"/>
-      <child link="${robot_namespace}/${prefix}_stator"/>
+    <joint name="tilt_to_${prefix}_estator" type="fixed">
+      <axis xyz="0 0 0"/>
+      <limit effort="1000.0" lower="0.0" upper="0.00" velocity="0.5"/>
+      <parent link="${parent}"/>
+      <child link="${prefix}_stator"/>
+    </joint>
+    <!--
+    <joint name="tilt_to_${prefix}_estator" type="revolute">
+      <axis xyz="0 ${reflect*1} 0"/>
+      <limit effort="1000.0" lower="0.0" upper="0.00" velocity="0.5"/>
+      <parent link="${parent}"/>
+      <child link="${prefix}_stator"/>
       <origin xyz="0 0 0"/>
     </joint>
-    <gazebo reference="${robot_namespace}/${prefix}_stator">
+    <transmission name="${prefix}_estator_trans" type="SimpleTransmission">
+      <type>transmission_interface/SimpleTransmission</type>
+      <actuator name="${prefix}_estator_motor">
+        <mechanicalReduction>1</mechanicalReduction>
+      </actuator>
+      <joint name="tilt_to_${prefix}_estator">
+        <hardwareInterface>hardware_interface/PositionJointInterface</hardwareInterface>
+      </joint>
+    </transmission>
+    -->
+    <gazebo reference="${prefix}_stator">
       <material>Gazebo/${color}</material>
     </gazebo>
   </xacro:macro>
-  <!--XACRO DO IMU : joint , link , sensor
+  <!--MACRO PARA CRIACAO DO ROTOR -->
+  <xacro:macro name="vertical_rotor" params="prefix direction motor_constant moment_constant parent mass_rotor radius_rotor time_constant_up time_constant_down max_rot_velocity motor_number rotor_drag_coefficient rolling_moment_coefficient color mesh mesh_scale *origin *inertia">
+    <!-- -->
+    <joint name="${prefix}_rotor_joint" type="fixed">
+      <xacro:insert_block name="origin" />
+      <parent link="${parent}" />
+      <child link="${prefix}_rotor" />
+    </joint>
+    <link name="${prefix}_rotor">
+      <inertial>
+        <mass value="${mass_rotor}" /> <!-- [kg] -->
+        <xacro:insert_block name="inertia" />
+      </inertial>
+      <visual>
+        <geometry>
+          <mesh filename="package://bicopter_sim/bicopter_description/meshes/${mesh}_${direction}.dae" scale="${mesh_scale}" />
+        </geometry>
+      </visual>
+      <collision>
+        <geometry>
+          <cylinder length="0.005" radius="${radius_rotor}" /> <!-- [m] -->
+        </geometry>
+      </collision>
+    </link>
+     <!-- Rotor joint and link
+    <joint name="${prefix}_rotor_joint" type="continuous">
+      <xacro:insert_block name="origin" />
+      <axis xyz="0 0 1" />
+      <limit effort="1000" velocity="1.0"/>
+      <parent link="${parent}" />
+      <child link="${prefix}_rotor" />
+    </joint>
+    <transmission name="${prefix}_motor_trans" type="SimpleTransmission">
+      <type>transmission_interface/SimpleTransmission</type>
+      <actuator name="${prefix}_motor">
+        <mechanicalReduction>1</mechanicalReduction>
+      </actuator>
+      <joint name="${prefix}_rotor_joint">
+        <hardwareInterface>hardware_interface/PositionJointInterface</hardwareInterface>
+      </joint>
+    </transmission>
+    -->
+    <!--
+    <gazebo>
+      <plugin name="${prefix}_motor_model" filename="librotors_gazebo_motor_model.so">
+        <jointName>${prefix}_rotor_joint</jointName>
+        <linkName>${prefix}_rotor</linkName>
+        <turningDirection>${direction}</turningDirection>
+        <timeConstantUp>${time_constant_up}</timeConstantUp>
+        <timeConstantDown>${time_constant_down}</timeConstantDown>
+        <maxRotVelocity>${max_rot_velocity}</maxRotVelocity>
+        <motorConstant>${motor_constant}</motorConstant>
+        <momentConstant>${moment_constant}</momentConstant>
+        <commandSubTopic>gazebo/command/motor_speed</commandSubTopic>
+        <motorNumber>${motor_number}</motorNumber>
+        <rotorDragCoefficient>${rotor_drag_coefficient}</rotorDragCoefficient>
+        <rollingMomentCoefficient>${rolling_moment_coefficient}</rollingMomentCoefficient>
+        <motorSpeedPubTopic>motor_speed/${prefix}</motorSpeedPubTopic>
+        <rotorVelocitySlowdownSim>${rotor_velocity_slowdown_sim}</rotorVelocitySlowdownSim>
+      </plugin>
+    </gazebo>
+     -->
+    <gazebo reference="${prefix}_rotor">
+      <material>Gazebo/${color}</material>
+    </gazebo>
+    </xacro:macro>
+ </robot>
+ <!--XACRO DO IMU : joint , link , sensor
   <xacro:macro name="imu_sensor" params="xyz rpy parent">
     <link name="imu_sensor_link">
@@ -272,54 +366,2 @@
    <xacro:imu_sensor xyz="0 0.05 0" rpy="0 0 0" parent="base_link" />
    -->
-  <!--MACRO PARA CRIACAO DO ROTOR -->
-  <xacro:macro name="vertical_rotor" params="robot_namespace suffix direction motor_constant moment_constant parent mass_rotor radius_rotor time_constant_up time_constant_down max_rot_velocity motor_number rotor_drag_coefficient rolling_moment_coefficient color mesh mesh_scale *origin *inertia">
-    <!-- Rotor joint and link  -->
-    <joint name="${robot_namespace}/rotor_${motor_number}_joint" type="continuous">
-      <xacro:insert_block name="origin" />
-      <axis xyz="0 0 1" />
-      <parent link="${parent}" />
-      <child link="${robot_namespace}/rotor_${motor_number}" />
-    </joint>
-    <!-- TODO(ff): not currently set because it's not yet supported -->
-    <!-- <gazebo reference="rotor_${motor_number}_joint"> <axis> <xyz>0 0 1</xyz>
-      <limit> <velocity> ${max_rot_velocity} </velocity> </limit> </axis> </gazebo> -->
-    <link name="${robot_namespace}/rotor_${motor_number}">
-      <inertial>
-        <mass value="${mass_rotor}" /> <!-- [kg] -->
-        <xacro:insert_block name="inertia" />
-      </inertial>
-      <visual>
-        <geometry>
-          <mesh filename="package://bicopter_sim/bicopter_description/meshes/${mesh}_${direction}.dae" scale="${mesh_scale}" />
-        </geometry>
-      </visual>
-      <collision>
-        <geometry>
-          <cylinder length="0.005" radius="${radius_rotor}" /> <!-- [m] -->
-        </geometry>
-      </collision>
-    </link>
-    <gazebo>
-      <plugin name="${robot_namespace}_${suffix}_motor_model" filename="librotors_gazebo_motor_model.so">
-        <robotNamespace>${robot_namespace}</robotNamespace>
-        <jointName>rotor_${motor_number}_joint</jointName>
-        <linkName>rotor_${motor_number}</linkName>
-        <turningDirection>${direction}</turningDirection>
-        <timeConstantUp>${time_constant_up}</timeConstantUp>
-        <timeConstantDown>${time_constant_down}</timeConstantDown>
-        <maxRotVelocity>${max_rot_velocity}</maxRotVelocity>
-        <motorConstant>${motor_constant}</motorConstant>
-        <momentConstant>${moment_constant}</momentConstant>
-        <commandSubTopic>gazebo/command/motor_speed</commandSubTopic>
-        <motorNumber>${motor_number}</motorNumber>
-        <rotorDragCoefficient>${rotor_drag_coefficient}</rotorDragCoefficient>
-        <rollingMomentCoefficient>${rolling_moment_coefficient}</rollingMomentCoefficient>
-        <motorSpeedPubTopic>motor_speed/${motor_number}</motorSpeedPubTopic>
-        <rotorVelocitySlowdownSim>${rotor_velocity_slowdown_sim}</rotorVelocitySlowdownSim>
-      </plugin>
-    </gazebo>
-    <gazebo reference="${robot_namespace}/rotor_${motor_number}">
-      <material>Gazebo/${color}</material>
-    </gazebo>
-    </xacro:macro>
- </robot>
